File: KiCad/rev2a/ec1834-post.sch (KiCad schematic (older format))
At the start: 29 parts, among them J0 BUS_EC1834_8Bit, J1 Bus_ISA_8bit, J2 Conn_02x07_Odd_Even, J3 Conn_01x03, J4 Conn_02x06_Odd_Even, SW1 SW_DIP_x10, U1 74LS688, U2 74LS86, U3 7432, U4 74HC374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

Commit message: Updated scheme to rev2 Update EPROM binaries Updated PCB to rev2 and new foot prints Added better documentation
Parts:
- removed R4, R5: 10k, Resistor_THT:R_Axial_DIN0207_L6.3mm_D2.5mm_P10.16mm_Horizontal, symbol Device:R
- removed RN1: R_Network08, Resistor_THT:R_Array_SIP9, symbol Device:R_Network08
- added RN1: R_Network10, Resistor_THT:R_Array_SIP11, symbol Device:R_Network10
- J0: symbol ec1834-post-lib:BUS_EC1834_8Bit -> ec1834-post-rescue:BUS_EC1834_8Bit-ec1834-post-lib
- U5, U6: symbol ec1834-post-lib:2732 -> ec1834-post-rescue:2732-ec1834-post-lib
Connections:
- wire segments 300 -> 295
- no-connect marks 78 -> 79
Other:
- note added: "disconnect U2.11 and U3.9\nconnect U3.9 to GND\n\nDisplay will work for A0-9 (IO 0x00 to 0x3ff)\nLogic Analyzer will work for A0-9\nIOR/IOW via output pins"
- moved on the sheet: R3, U2A, U2B, U2C, U2D, U2E, U3D
