File: KiCad/rev2b/ec1834-post.kicad_pcb (KiCad board)
At the start: 2 copper layers, 116.9 x 103.7 mm, 37 parts, among them J0 BUS_EC1834_8Bit, J1 Bus_ISA_8bit, J2 Conn_02x07_Odd_Even, J3 Conn_01x03, J4 Conn_02x06_Odd_Even, Q1 BC337, Q2 BC337, SW1 SW_DIP_x10, U1 74LS688, U2 74LS86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

Commit message: Fixed schematics and PCB (RN2-RN5 value changed to 1K5 R) Added an image Added german documentation
Parts:
- RN2, RN3, RN4, RN5: value 330 -> 1500
