File: KiCad/rev2b/ec1834-post.sch (KiCad schematic (older format))
At the start: 29 parts, among them J0 BUS_EC1834_8Bit, J1 Bus_ISA_8bit, J2 Conn_02x07_Odd_Even, J3 Conn_01x03, J4 Conn_02x06_Odd_Even, SW1 SW_DIP_x10, U1 74LS688, U2 74LS86, U3 7432, U4 74HC374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

Commit message: Updated scheme to rev2 Update EPROM binaries Updated PCB to rev2 and new foot prints Added better documentation
Parts:
- removed R1, R2: 470, Resistor_THT:R_Axial_DIN0207_L6.3mm_D2.5mm_P10.16mm_Horizontal, symbol Device:R
- added Q1, Q2: BC337, Package_TO_SOT_THT:TO-92_Inline, symbol Transistor_BJT:BC337
- added R4, R5: 1k, Resistor_THT:R_Axial_DIN0207_L6.3mm_D2.5mm_P10.16mm_Horizontal, symbol Device:R
- added R6: 220, Resistor_THT:R_Axial_DIN0207_L6.3mm_D2.5mm_P10.16mm_Horizontal, symbol Device:R
- added RN2, RN3, RN4, RN5: 330, Resistor_THT:R_Array_SIP8, symbol Device:R_Pack04_SIP
- J0: footprint Connector_DIN:DIN41612_C_2x32_Male_Horizontal_THT -> Connector_DIN:DIN41612_C_3x32_Male_Horizontal_THT; symbol ec1834-post-lib:BUS_EC1834_8Bit -> ec1834-post-rescue:BUS_EC1834_8Bit-ec1834-post-lib
- RN1: value R_Network08 -> SIL9-8 10K
- U5, U6: symbol ec1834-post-lib:2732 -> ec1834-post-rescue:2732-ec1834-post-lib
- renumbered R3 to R1, R4 to R2, R5 to R3
Connections:
- wire segments 300 -> 363
- no-connect marks 78 -> 83
Other:
- moved on the sheet: J2, J3, J4, R1, U2A, U2B, U2C, U2D, U2E, U3A, U7, U8

Commit message: Some schematics beautify actions Added schematics as PNG Typo fixed in BOM
Other:
- note added: "The display used by myself is a TDSR3150.\nIt is placed with dot down, when DIN slot is viewed on bottom.\nThe user will see it reversed. EPROM content reverses the output"
- moved on the sheet: C1, C2, C3, C4, C5, C6, C7, C8, J0, J1, Q1, Q2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

Commit message: Fixed schematics and PCB (RN2-RN5 value changed to 1K5 R) Added an image Added german documentation
Parts:
- RN2, RN3, RN4, RN5: value 330 -> 1500
Other:
- note added: "Das Display, welches ich nutze, ist ein TDSR3150.\nEs wird verkehrt herum eingbaut. Der Punkt ist auf Seite des DIN Slots.\nDie Ansicht wird im EPROM um 180° gedreht, so dass der Nutzer es ablesen kann."
- note added: "U1 verbindet die Adressfreigabe, AEN sowie IOW/IOR\nNur wenn das Signal Low Pegel hat, wird der Latch aktiviert und übernimmt die Daten vom Bus."
Changed lines of the file:
@@
 P 13000 6050
 F 0 "RN2" V 12958 6254 50  0000 L CNN
-F 1 "330" V 13049 6254 50  0000 L CNN
+F 1 "1500" V 13049 6254 50  0000 L CNN
 F 2 "Resistor_THT:R_Array_SIP8" V 13675 6050 50  0001 C CNN
 F 3 "http://www.vishay.com/docs/31509/csc.pdf" H 13000 6050 50  0001 C CNN
@@
 P 13000 7200
 F 0 "RN3" V 12958 7404 50  0000 L CNN
-F 1 "330" V 13049 7404 50  0000 L CNN
+F 1 "1500" V 13049 7404 50  0000 L CNN
 F 2 "Resistor_THT:R_Array_SIP8" V 13675 7200 50  0001 C CNN
 F 3 "http://www.vishay.com/docs/31509/csc.pdf" H 13000 7200 50  0001 C CNN
@@
 P 13000 3450
 F 0 "RN4" V 12958 3654 50  0000 L CNN
-F 1 "330" V 13049 3654 50  0000 L CNN
+F 1 "1500" V 13049 3654 50  0000 L CNN
 F 2 "Resistor_THT:R_Array_SIP8" V 13675 3450 50  0001 C CNN
 F 3 "http://www.vishay.com/docs/31509/csc.pdf" H 13000 3450 50  0001 C CNN
@@
 P 13000 4600
 F 0 "RN5" V 12958 4804 50  0000 L CNN
-F 1 "330" V 13049 4804 50  0000 L CNN
+F 1 "1500" V 13049 4804 50  0000 L CNN
 F 2 "Resistor_THT:R_Array_SIP8" V 13675 4600 50  0001 C CNN
 F 3 "http://www.vishay.com/docs/31509/csc.pdf" H 13000 4600 50  0001 C CNN
@@
 Wire Wire Line
 	14150 3750 14150 3850
+Text Notes 12600 1900 0    50   ~ 0
+Das Display, welches ich nutze, ist ein TDSR3150.\nEs wird verkehrt herum eingbaut. Der Punkt ist auf Seite des DIN Slots.\nDie Ansicht wird im EPROM um 180° gedreht, so dass der Nutzer es ablesen kann.
+Text Notes 7550 2350 0    50   ~ 0
+U1 verbindet die Adressfreigabe, AEN sowie IOW/IOR\nNur wenn das Signal Low Pegel hat, wird der Latch aktiviert und übernimmt die Daten vom Bus.
 $EndSCHEMATC
